Commit message: Add files via upload

File: my_bot/urdf/inno.xacro (robot description, xacro)
@@ -1,10 +1,10 @@
 <?xml version="1.0" ?>
 <robot name="inno" xmlns:xacro="http://www.ros.org/wiki/xacro">
-<xacro:include filename="$(find my_bot)/urdf/inno.gazebo" />
+<!--<xacro:include filename="$(find my_bot)/urdf/inno.gazebo" /> -->
 <xacro:include filename="$(find my_bot)/urdf/robo_control.xacro" />
-<xacro:property name="base_width" value="0.31"/>
+<xacro:property name="base_width" value="0.38"/>
 <xacro:property name="base_length" value="0.42"/>
 <xacro:property name="base_height" value="0.18"/>
-<xacro:property name="wheel_radius" value="0.10"/>
+<xacro:property name="wheel_radius" value="0.11"/>
 <xacro:property name="wheel_width" value="0.04"/>
 <xacro:property name="wheel_ygap" value="0.025"/>

File: my_bot/urdf/robo_control.xacro (robot description, xacro)
@@ -7,6 +7,6 @@
             <right_joint>drivewhl_r_joint</right_joint>
             <!-- kinematics -->
-            <wheel_separation>0.2</wheel_separation>
-            <wheel_diameter>0.14</wheel_diameter>
+            <wheel_separation>0.42</wheel_separation>
+            <wheel_diameter>0.22</wheel_diameter>
             <!-- limits -->
             <max_wheel_torque>200</max_wheel_torque>
